File: Power_Delivery_Board/Power_Delivery_Board.kicad_pcb (KiCad board)
At the start: 2 copper layers, 52.9 x 41.9 mm, 48 parts, among them IC1 STUSB4500QTR, J1 USB C, J2 IO pins, J3 Power Output, J4 IO Pins, J5 Qwiic, Q1 STL6P3LLH6

Commit message: Correcciones finales
Parts:
- added G***: LOGO, LOGO:logo, B.Cu at (167.3, 69.8)
- moved REF** 2.62 mm to (158.0, 68.0) (x2)
- renumbered D7 to Power_ok2, D6 to Power_ok3, D8 to gpio
Routing:
- net GND: track 114.3 -> 117.3 mm
- net /D+: track 27.6 -> 28.7 mm
- net /D-: track 31.2 -> 32.1 mm
- net /SCL: track 38.3 -> 39.1 mm
Other:
- board size 52.9 x 41.9 mm -> 53 x 45 mm
- board text added: "Errores DRC aprobados: - Pad near pad: @(129.602mm, 79.822mm) Pad S1 on F.Cu Internal, Non-copper of J1 @(130.852mm, 79.292mm) Pad on F.Cu, B.Cu Internal, Non-copper of J1 - Pad near pad: @(150.876mm, 77.440mm) Pad 2 on B.Cu Non-copper of J1 @(150.876mm, 78.740mm) Pad 1 on B.Cu, Non-copper of J1 - Pad near pad: @(151.832mm, 89.916mm) Pad 1 on B.Cu Non-copper of J1 @(153.132mm, 89.916mm) Pad 2 on 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"
- board text added: "Grilla 0.1270mm Margen 1mm"
- board text added: "IND. ARG."
- board text added: "POWER"
- board text added: "Pads 1mm Agujeros 0.5mm"
- board text added: "Pistas (por defecto) - ancho 0.2mm -margen 0.18mm Pistas (VCC VDD GND) - ancho 0.8mm -margen 0.3mm"
- board text added: "Replica SparkFun Power Delivery Board V0.2 8/5/2021"
- board text added: "Terminación superficial: HASL"
- board text removed: "(por defecto) - pads 0.8mm - agujeros 0.4mm (VCC VDD GND) -pads 1.27 - agujeros 0.7mm"
- board text removed: "pistas (por defecto) - ancho 0.2mm -margen 0.18mm pistas (VCC VDD GND) - ancho 0.8mm -margen 0.3mm"
